Commit message: remove xacros files

File: src/robot_description/config/robot/robot.urdf.xacro (robot description, xacro)
@@ -2,6 +2,4 @@
 <robot name="robot"
   xmlns:xacro="http://www.ros.org/wiki/xacro">
-  <xacro:include filename="$(find robot_description)/config/urdf/macros/link_geometry.urdf.xacro" />
-  <xacro:include filename="$(find robot_description)/config/urdf/macros/properties_robot.urdf.xacro" />
   <xacro:include filename="$(find robot_description)/config/urdf/macros/parts/base_robot.urdf.xacro" />
   <xacro:include filename="$(find robot_description)/config/urdf/macros/parts/rplidar_s2.urdf.xacro"/>

File: src/robot_description/config/urdf/macros/parts/base_robot.urdf.xacro (robot description, xacro)
@@ -11,16 +11,4 @@
       <child link="${name}"/>
     </joint>
-    <!-- joint: base -> right_motor -->
-    <joint name="${name}_to_right_motor" type="fixed">
-      <origin xyz="${ 0.42/2 - 0.075 } ${-(base_motor_lenght/2 + base_motor_gap/2)} ${0.03-base_motor_diameter/2}" rpy="${-PI/2} 0 0"/>
-      <parent link="${name}"/>
-      <child link="right_motor"/>
-    </joint>
-    <!-- joint: base -> left_motor -->
-    <joint name="${name}_to_left_motor" type="fixed">
-      <origin xyz="${ 0.42/2 - 0.075 } ${(base_motor_lenght/2 + base_motor_gap/2)} ${0.03-base_motor_diameter/2}" rpy="${-PI/2} 0 0"/>
-      <parent link="${name}"/>
-      <child link="left_motor"/>
-    </joint>
     <!-- joint: right_motor -> right_wheel -->
     <joint name="right_motor_to_right_wheel" type="continuous">
@@ -28,4 +16,18 @@
       <parent link="right_motor"/>
       <child link="right_wheel"/>
+      <axis xyz="0 0 1"/>
+    </joint>
+    <!-- joint: left_motor -> left_wheel -->
+    <joint name="left_motor_to_left_wheel" type="continuous">
+      <origin xyz="0 0 ${(base_wheel_lenght/2 + base_motor_lenght/2 + base_wheel_gap2base) }" rpy="0 0 0"/>
+      <parent link="left_motor"/>
+      <child link="left_wheel"/>
+      <axis xyz="0 0 1"/>
+    </joint>
+    <!-- joint: left_motor -> left_wheel -->
+    <joint name="left_motor_to_left_wheel" type="continuous">
+      <origin xyz="0 0 ${(base_wheel_lenght/2 + base_motor_lenght/2 + base_wheel_gap2base) }" rpy="0 0 0"/>
+      <parent link="left_motor"/>
+      <child link="left_wheel"/>
       <axis xyz="0 0 1"/>
     </joint>
