Commit message: Update robot_core.xacro

File: src/navtech/robot_description/description/robot_core.xacro (robot description, xacro)
@@ -1,5 +1,5 @@
 <?xml version="1.0"?>
 <robot xmlns:xacro="http://www.ros.org/wiki/xacro">
-    <!-- colors -->
+    <!-- ######## COLORS ######## -->
     <material name="white">
         <color rgba="1 1 1 1" />
@@ -17,12 +17,15 @@
         <color rgba="1 0 0 1"/>
     </material>
-    <!-- base link -->
+    <!-- BASE LINK-->
     <link name="base_link">
     </link>
+    <!-- ######## CHASSIS ######## -->
+    <!-- JOINT -->
     <joint name="chassis_joint" type="fixed">
         <parent link="base_link"/>
         <child link="chassis"/>
-        <origin xyz="-0.25 0 0"/>
+        <origin xyz="0 0 0"/>
     </joint>
+    <!-- LINK -->
     <link name="chassis">
         <visual>
@@ -34,3 +37,39 @@
         </visual>
     </link>
+    <!-- ######## LEFT WHEEL ######## -->
+    <!-- JOINT -->
+    <joint name="left_wheel_joint" type="continuous">
+        <parent link="base_link"/>
+        <child link="left_wheel"/>
+        <origin xyz="0 0.125 0" rpy="${pi/2} 0 0"/>
+        <axis xyz="0 0 1"/>
+    </joint>
+    <!-- LINK -->
+    <link name="left_wheel">
+        <visual>
+            <origin xyz="0 0 0" rpy="0 0 0"/>
+            <geometry>
+                <cylinder radius="0.05" length="0.01"/>
+            </geometry>
+            <material name="blue"/>
+        </visual>
+    </link>
+    <!-- ######## RIGHT WHEEL ######## -->
+    <!-- JOINT -->
+    <joint name="right_wheel_joint" type="continuous">
+        <parent link="base_link"/>
+        <child link="right_wheel"/>
+        <origin xyz="0 -0.125 0" rpy="${pi/2} 0 0"/>
+        <axis xyz="0 0 -1"/>
+    </joint>
+    <!-- LINK -->
+    <link name="right_wheel">
+        <visual>
+            <origin xyz="0 0 0" rpy="0 0 0"/>
+            <geometry>
+                <cylinder radius="0.05" length="0.01"/>
+            </geometry>
+            <material name="blue"/>
+        </visual>
+    </link>
 </robot>

Commit message: Update robot_core.xacro

File: src/navtech/robot_description/description/robot_core.xacro (robot description, xacro)
@@ -37,14 +37,14 @@
         </visual>
     </link>
-    <!-- ######## LEFT WHEEL ######## -->
+    <!-- ######## LEFT FRONT WHEEL ######## -->
     <!-- JOINT -->
-    <joint name="left_wheel_joint" type="continuous">
+    <joint name="left_front_wheel_joint" type="continuous">
         <parent link="base_link"/>
-        <child link="left_wheel"/>
-        <origin xyz="0 0.125 0" rpy="${pi/2} 0 0"/>
+        <child link="left_front_wheel"/>
+        <origin xyz="0.125 0.125 0" rpy="${pi/2} 0 0"/>
         <axis xyz="0 0 1"/>
     </joint>
     <!-- LINK -->
-    <link name="left_wheel">
+    <link name="left_front_wheel">
         <visual>
             <origin xyz="0 0 0" rpy="0 0 0"/>
@@ -55,14 +55,50 @@
         </visual>
     </link>
-    <!-- ######## RIGHT WHEEL ######## -->
+    <!-- ######## RIGHT FRONT WHEEL ######## -->
     <!-- JOINT -->
-    <joint name="right_wheel_joint" type="continuous">
+    <joint name="right_front_wheel_joint" type="continuous">
         <parent link="base_link"/>
-        <child link="right_wheel"/>
-        <origin xyz="0 -0.125 0" rpy="${pi/2} 0 0"/>
+        <child link="right_front_wheel"/>
+        <origin xyz="0.125 -0.125 0" rpy="${pi/2} 0 0"/>
         <axis xyz="0 0 -1"/>
     </joint>
     <!-- LINK -->
-    <link name="right_wheel">
+    <link name="right_front_wheel">
+        <visual>
+            <origin xyz="0 0 0" rpy="0 0 0"/>
+            <geometry>
+                <cylinder radius="0.05" length="0.01"/>
+            </geometry>
+            <material name="blue"/>
+        </visual>
+    </link>
+    <!-- ######## LEFT REAR WHEEL ######## -->
+    <!-- JOINT -->
+    <joint name="left_rear_wheel_joint" type="continuous">
+        <parent link="base_link"/>
+        <child link="left_rear_wheel"/>
+        <origin xyz="-0.125 0.125 0" rpy="${pi/2} 0 0"/>
+        <axis xyz="0 0 1"/>
+    </joint>
+    <!-- LINK -->
+    <link name="left_rear_wheel">
+        <visual>
+            <origin xyz="0 0 0" rpy="0 0 0"/>
+            <geometry>
+                <cylinder radius="0.05" length="0.01"/>
+            </geometry>
+            <material name="blue"/>
+        </visual>
+    </link>
+    <!-- ######## RIGHT REAR WHEEL ######## -->
+    <!-- JOINT -->
+    <joint name="right_rear_wheel_joint" type="continuous">
+        <parent link="base_link"/>
+        <child link="right_rear_wheel"/>
+        <origin xyz="-0.125 -0.125 0" rpy="${pi/2} 0 0"/>
+        <axis xyz="0 0 -1"/>
+    </joint>
+    <!-- LINK -->
+    <link name="right_rear_wheel">
         <visual>
             <origin xyz="0 0 0" rpy="0 0 0"/>

Commit message: Update robot_core.xacro

File: src/navtech/robot_description/description/robot_core.xacro (robot description, xacro)
@@ -37,14 +37,14 @@
         </visual>
     </link>
-    <!-- ######## LEFT FRONT WHEEL ######## -->
+    <!-- ######## LEFT WHEEL ######## -->
     <!-- JOINT -->
-    <joint name="left_front_wheel_joint" type="continuous">
+    <joint name="left_wheel_joint" type="continuous">
         <parent link="base_link"/>
-        <child link="left_front_wheel"/>
-        <origin xyz="0.125 0.125 0" rpy="${pi/2} 0 0"/>
+        <child link="left_wheel"/>
+        <origin xyz="0 0.125 0" rpy="${pi/2} 0 0"/>
         <axis xyz="0 0 1"/>
     </joint>
     <!-- LINK -->
-    <link name="left_front_wheel">
+    <link name="left_wheel">
         <visual>
             <origin xyz="0 0 0" rpy="0 0 0"/>
@@ -55,14 +55,14 @@
         </visual>
     </link>
-    <!-- ######## RIGHT FRONT WHEEL ######## -->
+    <!-- ######## RIGHT WHEEL ######## -->
     <!-- JOINT -->
-    <joint name="right_front_wheel_joint" type="continuous">
+    <joint name="right_wheel_joint" type="continuous">
         <parent link="base_link"/>
-        <child link="right_front_wheel"/>
-        <origin xyz="0.125 -0.125 0" rpy="${pi/2} 0 0"/>
+        <child link="right_wheel"/>
+        <origin xyz="0 -0.125 0" rpy="${pi/2} 0 0"/>
         <axis xyz="0 0 -1"/>
     </joint>
     <!-- LINK -->
-    <link name="right_front_wheel">
+    <link name="right_wheel">
         <visual>
             <origin xyz="0 0 0" rpy="0 0 0"/>
@@ -73,14 +73,14 @@
         </visual>
     </link>
-    <!-- ######## LEFT REAR WHEEL ######## -->
+    <!-- ######## FRONT WHEEL ######## -->
     <!-- JOINT -->
-    <joint name="left_rear_wheel_joint" type="continuous">
+    <joint name="front_wheel_joint" type="continuous">
         <parent link="base_link"/>
-        <child link="left_rear_wheel"/>
-        <origin xyz="-0.125 0.125 0" rpy="${pi/2} 0 0"/>
+        <child link="front_wheel"/>
+        <origin xyz="0.125 0 0" rpy="0 ${pi/2} 0"/>
         <axis xyz="0 0 1"/>
     </joint>
     <!-- LINK -->
-    <link name="left_rear_wheel">
+    <link name="front_wheel">
         <visual>
             <origin xyz="0 0 0" rpy="0 0 0"/>
@@ -91,14 +91,14 @@
         </visual>
     </link>
-    <!-- ######## RIGHT REAR WHEEL ######## -->
+    <!-- ######## BACK WHEEL ######## -->
     <!-- JOINT -->
-    <joint name="right_rear_wheel_joint" type="continuous">
+    <joint name="back_wheel_joint" type="continuous">
         <parent link="base_link"/>
-        <child link="right_rear_wheel"/>
-        <origin xyz="-0.125 -0.125 0" rpy="${pi/2} 0 0"/>
-        <axis xyz="0 0 -1"/>
+        <child link="back_wheel"/>
+        <origin xyz="-0.125 0 0" rpy="0 ${pi/2} 0"/>
+        <axis xyz="0 0 1"/>
     </joint>
     <!-- LINK -->
-    <link name="right_rear_wheel">
+    <link name="back_wheel">
         <visual>
             <origin xyz="0 0 0" rpy="0 0 0"/>

Commit message: Update robot_core.xacro

File: src/navtech/robot_description/description/robot_core.xacro (robot description, xacro)
@@ -29,4 +29,55 @@
     <!-- LINK -->
     <link name="chassis">
+        <visual>
+            <origin xyz="0 0 0" rpy="0 0 0"/>
+            <geometry>
+                <cylinder radius="0.125" length="0.006"/>
+            </geometry>
+            <material name="white"/>
+        </visual>
+    </link>
+    <!-- ######## PLATFORM 1 ######## -->
+    <!-- JOINT -->
+    <joint name="platform1_joint" type="fixed">
+        <parent link="chassis"/>
+        <child link="platform1"/>
+        <origin xyz="0 0.07 0"/>
+    </joint>
+    <!-- LINK -->
+    <link name="platform1">
+        <visual>
+            <origin xyz="0 0 0" rpy="0 0 0"/>
+            <geometry>
+                <cylinder radius="0.125" length="0.006"/>
+            </geometry>
+            <material name="white"/>
+        </visual>
+    </link>
+    <!-- ######## PLATFORM 2 ######## -->
+    <!-- JOINT -->
+    <joint name="platform2_joint" type="fixed">
+        <parent link="chassis"/>
+        <child link="platform2"/>
+        <origin xyz="0 -0.07 0"/>
+    </joint>
+    <!-- LINK -->
+    <link name="platform2">
+        <visual>
+            <origin xyz="0 0 0" rpy="0 0 0"/>
+            <geometry>
+                <cylinder radius="0.125" length="0.006"/>
+            </geometry>
+            <material name="white"/>
+        </visual>
+    </link>
+    <!-- ######## PLATFORM 3 ######## -->
+    <!-- JOINT -->
+    <joint name="platform3_joint" type="fixed">
+        <parent link="chassis"/>
+        <child link="platform3"/>
+        <origin xyz="0 0.14 0"/>
+    </joint>
+    <!-- LINK -->
+    <link name="platform3">
         <visual>
             <origin xyz="0 0 0" rpy="0 0 0"/>

Commit message: Update robot_core.xacro

File: src/navtech/robot_description/description/robot_core.xacro (robot description, xacro)
@@ -32,56 +32,5 @@
             <origin xyz="0 0 0" rpy="0 0 0"/>
             <geometry>
-                <cylinder radius="0.125" length="0.006"/>
-            </geometry>
-            <material name="white"/>
-        </visual>
-    </link>
-    <!-- ######## PLATFORM 1 ######## -->
-    <!-- JOINT -->
-    <joint name="platform1_joint" type="fixed">
-        <parent link="chassis"/>
-        <child link="platform1"/>
-        <origin xyz="0 0.07 0"/>
-    </joint>
-    <!-- LINK -->
-    <link name="platform1">
-        <visual>
-            <origin xyz="0 0 0" rpy="0 0 0"/>
-            <geometry>
-                <cylinder radius="0.125" length="0.006"/>
-            </geometry>
-            <material name="white"/>
-        </visual>
-    </link>
-    <!-- ######## PLATFORM 2 ######## -->
-    <!-- JOINT -->
-    <joint name="platform2_joint" type="fixed">
-        <parent link="chassis"/>
-        <child link="platform2"/>
-        <origin xyz="0 -0.07 0"/>
-    </joint>
-    <!-- LINK -->
-    <link name="platform2">
-        <visual>
-            <origin xyz="0 0 0" rpy="0 0 0"/>
-            <geometry>
-                <cylinder radius="0.125" length="0.006"/>
-            </geometry>
-            <material name="white"/>
-        </visual>
-    </link>
-    <!-- ######## PLATFORM 3 ######## -->
-    <!-- JOINT -->
-    <joint name="platform3_joint" type="fixed">
-        <parent link="chassis"/>
-        <child link="platform3"/>
-        <origin xyz="0 0.14 0"/>
-    </joint>
-    <!-- LINK -->
-    <link name="platform3">
-        <visual>
-            <origin xyz="0 0 0" rpy="0 0 0"/>
-            <geometry>
-                <cylinder radius="0.125" length="0.006"/>
+                <mesh filename="file://$(find robot_description)/meshes/base.dae" />
             </geometry>
             <material name="white"/>
@@ -101,5 +50,5 @@
             <origin xyz="0 0 0" rpy="0 0 0"/>
             <geometry>
-                <cylinder radius="0.05" length="0.01"/>
+                <mesh filename="file://$(find robot_description)/meshes/wheel.dae" />
             </geometry>
             <material name="blue"/>
@@ -119,5 +68,5 @@
             <origin xyz="0 0 0" rpy="0 0 0"/>
             <geometry>
-                <cylinder radius="0.05" length="0.01"/>
+                <mesh filename="file://$(find robot_description)/meshes/wheel.dae" />
             </geometry>
             <material name="blue"/>
@@ -137,5 +86,5 @@
             <origin xyz="0 0 0" rpy="0 0 0"/>
             <geometry>
-                <cylinder radius="0.05" length="0.01"/>
+                <mesh filename="file://$(find robot_description)/meshes/wheel.dae" />
             </geometry>
             <material name="blue"/>
@@ -155,5 +104,5 @@
             <origin xyz="0 0 0" rpy="0 0 0"/>
             <geometry>
-                <cylinder radius="0.05" length="0.01"/>
+                <mesh filename="file://$(find robot_description)/meshes/wheel.dae" />
             </geometry>
             <material name="blue"/>

Commit message: working organized TFs

File: src/navtech/robot_description/description/robot_core.xacro (robot description, xacro)
@@ -32,5 +32,56 @@
             <origin xyz="0 0 0" rpy="0 0 0"/>
             <geometry>
-                <mesh filename="file://$(find robot_description)/meshes/base.dae" />
+                <cylinder radius="0.125" length="0.006"/>
+            </geometry>
+            <material name="white"/>
+        </visual>
+    </link>
+    <!-- ######## PLATFORM 1 ######## -->
+    <!-- JOINT -->
+    <joint name="platform1_joint" type="fixed">
+        <parent link="chassis"/>
+        <child link="platform1"/>
+        <origin xyz="0 0 0.07"/>
+    </joint>
+    <!-- LINK -->
+    <link name="platform1">
+        <visual>
+            <origin xyz="0 0 0" rpy="0 0 0"/>
+            <geometry>
+                <cylinder radius="0.125" length="0.006"/>
+            </geometry>
+            <material name="white"/>
+        </visual>
+    </link>
+    <!-- ######## PLATFORM 2 ######## -->
+    <!-- JOINT -->
+    <joint name="platform2_joint" type="fixed">
+        <parent link="chassis"/>
+        <child link="platform2"/>
+        <origin xyz="0 0 0.14"/>
+    </joint>
+    <!-- LINK -->
+    <link name="platform2">
+        <visual>
+            <origin xyz="0 0 0" rpy="0 0 0"/>
+            <geometry>
+                <cylinder radius="0.125" length="0.006"/>
+            </geometry>
+            <material name="white"/>
+        </visual>
+    </link>
+    <!-- ######## PLATFORM 3 ######## -->
+    <!-- JOINT -->
+    <joint name="platform3_joint" type="fixed">
+        <parent link="chassis"/>
+        <child link="platform3"/>
+        <origin xyz="0 0 0.21"/>
+    </joint>
+    <!-- LINK -->
+    <link name="platform3">
+        <visual>
+            <origin xyz="0 0 0" rpy="0 0 0"/>
+            <geometry>
+                <cylinder radius="0.125" length="0.006"/>
             </geometry>
             <material name="white"/>
@@ -50,5 +101,5 @@
             <origin xyz="0 0 0" rpy="0 0 0"/>
             <geometry>
-                <mesh filename="file://$(find robot_description)/meshes/wheel.dae" />
+                <cylinder radius="0.05" length="0.05"/>
             </geometry>
             <material name="blue"/>
@@ -68,5 +119,5 @@
             <origin xyz="0 0 0" rpy="0 0 0"/>
             <geometry>
-                <mesh filename="file://$(find robot_description)/meshes/wheel.dae" />
+                <cylinder radius="0.05" length="0.05"/>
             </geometry>
             <material name="blue"/>
@@ -86,5 +137,5 @@
             <origin xyz="0 0 0" rpy="0 0 0"/>
             <geometry>
-                <mesh filename="file://$(find robot_description)/meshes/wheel.dae" />
+                <cylinder radius="0.05" length="0.05"/>
             </geometry>
             <material name="blue"/>
@@ -104,5 +155,5 @@
             <origin xyz="0 0 0" rpy="0 0 0"/>
             <geometry>
-                <mesh filename="file://$(find robot_description)/meshes/wheel.dae" />
+                <cylinder radius="0.05" length="0.05"/>
             </geometry>
             <material name="blue"/>

Commit message: working organized TFs

File: src/navtech/robot_description/description/robot_core.xacro (robot description, xacro)
@@ -93,5 +93,5 @@
         <parent link="base_link"/>
         <child link="left_wheel"/>
-        <origin xyz="0 0.125 0" rpy="${pi/2} 0 0"/>
+        <origin xyz="0 0.145 0" rpy="${pi/2} 0 0"/>
         <axis xyz="0 0 1"/>
     </joint>
@@ -111,5 +111,5 @@
         <parent link="base_link"/>
         <child link="right_wheel"/>
-        <origin xyz="0 -0.125 0" rpy="${pi/2} 0 0"/>
+        <origin xyz="0 -0.145 0" rpy="${pi/2} 0 0"/>
         <axis xyz="0 0 -1"/>
     </joint>
@@ -129,5 +129,5 @@
         <parent link="base_link"/>
         <child link="front_wheel"/>
-        <origin xyz="0.125 0 0" rpy="0 ${pi/2} 0"/>
+        <origin xyz="0.145 0 0" rpy="0 ${pi/2} 0"/>
         <axis xyz="0 0 1"/>
     </joint>
@@ -147,5 +147,5 @@
         <parent link="base_link"/>
         <child link="back_wheel"/>
-        <origin xyz="-0.125 0 0" rpy="0 ${pi/2} 0"/>
+        <origin xyz="-0.145 0 0" rpy="0 ${pi/2} 0"/>
         <axis xyz="0 0 1"/>
     </joint>
