Commit message: working organized TFs

File: src/navtech/robot_description/description/core.xacro (robot description, xacro)
@@ -31,7 +31,7 @@
     <link name="chassis">
         <visual>
-            <origin xyz="0 0 0" rpy="0 0 0"/>
+            <origin xyz="0 0 0.105" rpy="0 0 0"/>
             <geometry>
-                <cylinder radius="0.125" length="0.006"/>
+                <cylinder radius="0.125" length="0.21"/>
             </geometry>
             <material name="white"/>
@@ -40,68 +40,17 @@
             <origin xyz="0 0 0" rpy="0 0 0"/>
             <geometry>
-                <cylinder radius="0.125" length="0.006"/>
+                <cylinder radius="0.125" length="0.21"/>
             </geometry>
         </collision>
-        <xacro:inertial_cylinder mass="0.5" length="0.006" radius="0.125">
+        <xacro:inertial_cylinder mass="0.5" length="0.21" radius="0.125">
             <origin xyz="0 0 0" rpy="0 0 0"/>
         </xacro:inertial_cylinder>
-    </link>
-    <!-- ######## PLATFORM 1 ######## -->
-    <!-- JOINT -->
-    <joint name="platform1_joint" type="fixed">
-        <parent link="chassis"/>
-        <child link="platform1"/>
-        <origin xyz="0 0 0.07"/>
-    </joint>
-    <!-- LINK -->
-    <link name="platform1">
-        <visual>
-            <origin xyz="0 0 0" rpy="0 0 0"/>
-            <geometry>
-                <cylinder radius="0.125" length="0.006"/>
-            </geometry>
-            <material name="white"/>
-        </visual>
-    </link>
-    <!-- ######## PLATFORM 2 ######## -->
-    <!-- JOINT -->
-    <joint name="platform2_joint" type="fixed">
-        <parent link="chassis"/>
-        <child link="platform2"/>
-        <origin xyz="0 0 0.14"/>
-    </joint>
-    <!-- LINK -->
-    <link name="platform2">
-        <visual>
-            <origin xyz="0 0 0" rpy="0 0 0"/>
-            <geometry>
-                <cylinder radius="0.125" length="0.006"/>
-            </geometry>
-            <material name="white"/>
-        </visual>
-    </link>
-    <!-- ######## PLATFORM 3 ######## -->
-    <!-- JOINT -->
-    <joint name="platform3_joint" type="fixed">
-        <parent link="chassis"/>
-        <child link="platform3"/>
-        <origin xyz="0 0 0.21"/>
-    </joint>
-    <!-- LINK -->
-    <link name="platform3">
-        <visual>
-            <origin xyz="0 0 0" rpy="0 0 0"/>
-            <geometry>
-                <cylinder radius="0.125" length="0.006"/>
-            </geometry>
-            <material name="white"/>
-        </visual>
     </link>
     <!-- ######## LEFT WHEEL ######## -->
     <!-- JOINT -->
     <joint name="left_wheel_joint" type="continuous">
-        <parent link="chassis"/>
+        <parent link="base_link"/>
         <child link="left_wheel"/>
-        <origin xyz="0 0.150 -0.015" rpy="${pi/2} 0 0"/>
+        <origin xyz="0 0.150 0" rpy="${pi/2} 0 0"/>
         <axis xyz="0 0 1"/>
     </joint>
@@ -125,10 +74,13 @@
         </xacro:inertial_cylinder>
     </link>
+    <gazebo reference="left_wheel">
+        <material>Gazebo/Blue</material>
+    </gazebo>
     <!-- ######## RIGHT WHEEL ######## -->
     <!-- JOINT -->
     <joint name="right_wheel_joint" type="continuous">
-        <parent link="chassis"/>
+        <parent link="base_link"/>
         <child link="right_wheel"/>
-        <origin xyz="0 -0.150 -0.015" rpy="${pi/2} 0 0"/>
+        <origin xyz="0 -0.150 0" rpy="${pi/2} 0 0"/>
         <axis xyz="0 0 -1"/>
     </joint>
@@ -152,10 +104,13 @@
         </xacro:inertial_cylinder>
     </link>
+    <gazebo reference="right_wheel">
+        <material>Gazebo/Blue</material>
+    </gazebo>
     <!-- ######## FRONT WHEEL ######## -->
     <!-- JOINT -->
     <joint name="front_wheel_joint" type="continuous">
-        <parent link="chassis"/>
+        <parent link="base_link"/>
         <child link="front_wheel"/>
-        <origin xyz="0.150 0 -0.015" rpy="0 ${pi/2} 0"/>
+        <origin xyz="0.150 0 0" rpy="0 ${pi/2} 0"/>
         <axis xyz="0 0 1"/>
     </joint>
@@ -179,10 +134,13 @@
         </xacro:inertial_cylinder>
     </link>
+    <gazebo reference="front_wheel">
+        <material>Gazebo/Blue</material>
+    </gazebo>
     <!-- ######## BACK WHEEL ######## -->
     <!-- JOINT -->
     <joint name="back_wheel_joint" type="continuous">
-        <parent link="chassis"/>
+        <parent link="base_link"/>
         <child link="back_wheel"/>
-        <origin xyz="-0.150 0 -0.015" rpy="0 ${pi/2} 0"/>
+        <origin xyz="-0.150 0 0" rpy="0 ${pi/2} 0"/>
         <axis xyz="0 0 1"/>
     </joint>
@@ -206,3 +164,6 @@
         </xacro:inertial_cylinder>
     </link>
+    <gazebo reference="back_wheel">
+        <material>Gazebo/Blue</material>
+    </gazebo>
 </robot>

File: src/navtech/robot_description/description/robot.urdf.xacro (robot description, xacro)
@@ -2,3 +2,4 @@
 <robot xmlns:xacro="http://www.ros.org/wiki/xacro"  name="robot">
     <xacro:include filename="core.xacro" />
+    <xacro:include filename="control.xacro" />
 </robot>

Commit message: add footprint

File: src/navtech/robot_description/description/core.xacro (robot description, xacro)
@@ -21,4 +21,11 @@
     <link name="base_link">
     </link>
+    <!-- FOOTPRINT -->
+    <link name='base_footprint'/>
+    <joint name="joint_base_footprint_to_base" type="fixed">
+      <origin xyz="0 0 0"/>
+      <parent link="base_footprint"/>
+      <child link="base"/>
+    </joint>
     <!-- ######## CHASSIS ######## -->
     <!-- JOINT -->

Commit message: working organized TFs

File: src/navtech/robot_description/description/core.xacro (robot description, xacro)
@@ -18,14 +18,15 @@
         <color rgba="1 0 0 1"/>
     </material>
-    <!-- BASE LINK-->
+    <!-- ######## BASE LINK ######## -->
     <link name="base_link">
     </link>
-    <!-- FOOTPRINT -->
-    <link name='base_footprint'/>
-    <joint name="joint_base_footprint_to_base" type="fixed">
-      <origin xyz="0 0 0"/>
-      <parent link="base_footprint"/>
-      <child link="base"/>
+    <!-- ######## BASE FOOTPRINT ######## -->
+    <joint name="base_footprint_joint" type="fixed">
+        <parent link="base_link"/>
+        <child link="base_footprint"/>
+        <origin xyz="0 0 0" rpy="0 0 0"/>
     </joint>
+    <link name="base_footprint">
+    </link>
     <!-- ######## CHASSIS ######## -->
     <!-- JOINT -->

File: src/navtech/robot_description/description/robot.urdf.xacro (robot description, xacro)
@@ -3,3 +3,4 @@
     <xacro:include filename="core.xacro" />
     <xacro:include filename="control.xacro" />
+    <xacro:include filename="sensors.xacro" />
 </robot>
