Commit message: create SLAM

File: src/navtech/robot/description/control.xacro (robot description, xacro)
@@ -2,12 +2,11 @@
 <robot xmlns:xacro="http://www.ros.org/wiki/xacro">
     <gazebo>
-        <plugin name="base_link_controller" filename="libgazebo_ros_planar_move.so">
+        <plugin name="object_controller" filename="libgazebo_ros_planar_move.so">
           <robotNamespace>/</robotNamespace>
           <commandTopic>cmd_vel</commandTopic>
           <odometryTopic>odom</odometryTopic>
           <odometryFrame>odom</odometryFrame>
-          <odometryRate>100</odometryRate>
-          <cmdTimeout>-1</cmdTimeout>
-          <robotBaseFrame>base_link</robotBaseFrame>
+          <odometryRate>20</odometryRate>
+          <robotBaseFrame>base_footprint</robotBaseFrame>
         </plugin>
     </gazebo>

File: src/navtech/robot/description/core.xacro (robot description, xacro)
@@ -22,11 +22,14 @@
     </link>
     <!-- ######## BASE FOOTPRINT ######## -->
-    <joint name="base_footprint_joint" type="fixed">
-        <parent link="base_link"/>
-        <child link="base_footprint"/>
-        <origin xyz="0 0 0" rpy="0 0 0"/>
+    <link name="base_footprint">
+        <visual>
+            <origin xyz="0 0 0" rpy="0 0 0" />
+        </visual>
+    </link>
+    <joint name="base_link_joint" type="fixed">
+        <origin xyz="0.0 0 0" rpy="0 0 0" />
+        <parent link="base_footprint"/>
+        <child link="base_link" />
     </joint>
-    <link name="base_footprint">
-    </link>
     <!-- ######## CHASSIS ######## -->
     <!-- JOINT -->

File: src/navtech/robot/description/sensors.xacro (robot description, xacro)
@@ -2,7 +2,7 @@
 <robot xmlns:xacro="http://www.ros.org/wiki/xacro" >
     <joint name="laser_joint" type="fixed">
-        <parent link="chassis"/>
+        <parent link="base_link"/>
         <child link="laser_frame"/>
-        <origin xyz="0 0 0.22" rpy="0 0 0"/>
+        <origin xyz="0 0 0.25" rpy="0 0 0"/>
     </joint>
     <link name="laser_frame">
